Commit message: redefined the mechanism to slider

File: dobot_ws/src/slider_description/urdf/common/slider_ros2_macro.xacro (robot description, xacro)
@@ -14,13 +14,18 @@
         </joint>
     </xacro:macro>
-    <xacro:macro name="vertical_lift_ros2_control" params="name lower upper">
+    <xacro:macro name="passive_joint_interface" params="joint_name initial:=0.0002">
+        <joint name="${joint_name}">
+            <state_interface name="position">
+                <param name="initial_value">${initial}</param>
+            </state_interface>
+            <state_interface name="velocity" />
+        </joint>
+    </xacro:macro>
+    <xacro:macro name="ros2_control_system" params="name **joint_interfaces">
         <ros2_control name="${name}" type="system">
             <hardware>
                 <plugin>gz_ros2_control/GazeboSimSystem</plugin>
             </hardware>
-            <xacro:prismatic_joint_interface joint_name="lift_mid_joint" lower="${lower}"
-                upper="${upper}" />
-            <xacro:prismatic_joint_interface joint_name="lift_top_joint" lower="${lower}"
-                upper="${upper}" />
+            <xacro:insert_block name="joint_interfaces" />
         </ros2_control>
     </xacro:macro>
